File: example.brd (EAGLE design)
At the start: 40.6 x 35.6 mm, 6 parts

Commit message: Removed showing pin names for symbol. Updated example
Parts:
- moved FID1 2.54 mm to (5.08, 34.3)
- moved LOGO2 2.54 mm to (2.54, 6.86)
- moved U$2 2.54 mm to (0.00, 0.00)
- moved FID2 2.54 mm to (35.6, 1.27)
- moved FID3 2.54 mm to (35.6, 34.3)
Other:
- board text added: "10cm x 10cm"
- board text added: "5cm x 5cm"
